Commit message: Enhance OnPolicyTrainer logging and refine URDF for robot simulation; add BipedalRobotEnv example

File: examples/mybot.urdf (robot description, URDF)
Before this commit: robot mybot, 20 links, 19 joints
Links:
- removed link camera
- link base_link: mass 1 -> 0.1
Joints:
- removed joint joint_camera_base_link
- joint joint_link10_link12: axis 0 0 1 -> (none); limit lower=-0.065 upper=0.565 effort=100 velocity=1 -> (none)
- joint joint_link13_link15: axis 0 0 1 -> (none); limit lower=-0.465 upper=0.165 effort=100 velocity=1 -> (none)
- joint joint_link14_link16: axis 0 0 1 -> (none); limit lower=-0.465 upper=0.165 effort=100 velocity=1 -> (none)
- joint joint_link5_link7: axis 0 0 1 -> (none); limit lower=-0.065 upper=0.565 effort=100 velocity=1 -> (none)
- joint joint_link6_link8: axis 0 0 1 -> (none); limit lower=-0.065 upper=0.565 effort=100 velocity=1 -> (none)
- joint joint_link9_link11: axis 0 0 1 -> (none); limit lower=-0.065 upper=0.565 effort=100 velocity=1 -> (none)

Commit message: Add example for Kullback-Leibler divergence with Product of Normals
- Implemented classes P_1, P_2, and Q as Normal distributions.
- Created a ProductOfNormal instance combining P_1 and P_2.
- Added KullbackLeibler loss calculation using the defined distributions.
- Included a print statement to display the KL divergence output.

File: examples/mybot.urdf (robot description, URDF)
Before this commit: robot mybot, 19 links, 18 joints
Links:
- added link camera, mass 0.1; visual box size=0.05 0.05 0.05
Joints:
- added joint joint_camera_base_link: type fixed, parent base_link, child camera, origin xyz=0 -0.25 0 rpy=0 0 0
